File: printer_mods/VinnyCordeiro/RGB_LED_grid_for_SB/KiCad/RGBW_LED_circular_panel_for_Stealthburner.kicad_sch (KiCad schematic)
At the start: 11 parts, among them J1 Conn_02x03_Odd_Even

Commit message: Updated PCB, solve need for inline resistor for impedance matching (#716)
* Create README.md

* Create README.md

* Update README.md

* Added KiCad project files

* Create README.md

* Added production files

* Update README.md

Added note on mixing RGB and RGBW LEDs.

* Update README.md

typo

* Create README.md

* Update README.md

Added VinnyCordeiro's RGB LED grid for Stealthburner

* Add files via upload

Animated GIF of the board working

* Update README.md

* Update README.md

* Update README.md

Added the KiCad version that was used to design the PCB

* Removed non-necessary components

Removed both the input resistor and the filtering capacitor, as they are not strictly necessary for this application.

* Delete bom.csv

* Delete cpl.csv

* Delete RGBW_LED_circular_panel_for_Stealthburner.zip

* Updated production files

* Update README.md
Parts:
- removed C1: 100nF, Capacitors_SMD:C_0402_NoSilk, symbol Device:C
- removed R1: 470R, Resistors_SMD:R_0402_NoSilk, symbol Device:R
Connections:
- net LED_IN: now also D1.4 (DIN)
Changed lines of the file:
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@@
-    (stroke (width 0) (type default) (color 0 0 0 0))
-  )
-  (wire (pts (xy 46.99 87.63) (xy 46.99 88.9))
     (stroke (width 0) (type default) (color 0 0 0 0))
   )
@@
     (stroke (width 0) (type default) (color 0 0 0 0))
   )
-  (wire (pts (xy 59.69 72.39) (xy 59.69 82.55))
+  (wire (pts (xy 59.69 63.5) (xy 59.69 82.55))
     (stroke (width 0) (type default) (color 0 0 0 0))
   )
@@
     (stroke (width 0) (type default) (color 0 0 0 0))
   )
-  (wire (pts (xy 59.69 63.5) (xy 59.69 64.77))
-    (stroke (width 0) (type default) (color 0 0 0 0))
-  )
   (wire (pts (xy 135.89 91.44) (xy 135.89 114.3))
     (stroke (width 0) (type default) (color 0 0 0 0))
@@
   )
   (wire (pts (xy 101.6 96.52) (xy 118.11 96.52))
-    (stroke (width 0) (type default) (color 0 0 0 0))
-  )
-  (wire (pts (xy 46.99 78.74) (xy 46.99 80.01))
     (stroke (width 0) (type default) (color 0 0 0 0))
   )
@@
     )
     (pin "1")
-  )
-  (symbol (lib_id "Device:C") (at 46.99 83.82 0) (unit 1)
-    (in_bom yes) (on_board yes)
-    (property "Reference" "C1" (id 0) (at 49.911 82.6516 0)
-      (effects (font (size 1.27 1.27)) (justify left))
-    )
-    (property "Value" "100nF" (id 1) (at 49.911 84.963 0)
-      (effects (font (size 1.27 1.27)) (justify left))
-    )
-    (property "Footprint" "Capacitors_SMD:C_0402_NoSilk" (id 2) (at 47.9552 87.63 0)
-      (effects (font (size 1.27 1.27)) hide)
-    )
-    (property "Datasheet" "~" (id 3) (at 46.99 83.82 0)
-      (effects (font (size 1.27 1.27)) hide)
-    )
-    (pin "1")
-    (pin "2")
-  )
-  (symbol (lib_id "power:+5V") (at 46.99 78.74 0) (unit 1)
-    (in_bom yes) (on_board yes)
-    (property "Reference" "#PWR02" (id 0) (at 46.99 82.55 0)
-      (effects (font (size 1.27 1.27)) hide)
-    )
-    (property "Value" "+5V" (id 1) (at 47.371 74.3458 0))
-    (property "Footprint" "" (id 2) (at 46.99 78.74 0)
-      (effects (font (size 1.27 1.27)) hide)
-    )
-    (property "Datasheet" "" (id 3) (at 46.99 78.74 0)
-      (effects (font (size 1.27 1.27)) hide)
-    )
-    (pin "1")
-  )
-  (symbol (lib_id "power:GND") (at 46.99 88.9 0) (unit 1)
-    (in_bom yes) (on_board yes)
-    (property "Reference" "#PWR03" (id 0) (at 46.99 95.25 0)
-      (effects (font (size 1.27 1.27)) hide)
-    )
-    (property "Value" "GND" (id 1) (at 47.117 93.2942 0))
-    (property "Footprint" "" (id 2) (at 46.99 88.9 0)
-      (effects (font (size 1.27 1.27)) hide)
-    )
-    (property "Datasheet" "" (id 3) (at 46.99 88.9 0)
-      (effects (font (size 1.27 1.27)) hide)
-    )
-    (pin "1")
-  )
-  (symbol (lib_id "Device:R") (at 59.69 68.58 0) (unit 1)
-    (in_bom yes) (on_board yes)
-    (property "Reference" "R1" (id 0) (at 60.96 63.5 0)
-      (effects (font (size 1.27 1.27)) (justify left))
-    )
-    (property "Value" "470R" (id 1) (at 60.96 66.04 0)
-      (effects (font (size 1.27 1.27)) (justify left))
-    )
-    (property "Footprint" "Resistors_SMD:R_0402_NoSilk" (id 2) (at 57.912 68.58 90)
-      (effects (font (size 1.27 1.27)) hide)
-    )
-    (property "Datasheet" "~" (id 3) (at 59.69 68.58 0)
-      (effects (font (size 1.27 1.27)) hide)
-    )
-    (pin "1")
-    (pin "2")
   )
   (symbol (lib_id "Connector_Generic:Conn_02x03_Odd_Even") (at 161.29 102.87 0) (unit 1)
@@
       (reference "#PWR01") (unit 1) (value "+5V") (footprint "")
     )
-    (path "/00000000-0000-0000-0000-000061c83d5e"
-      (reference "#PWR02") (unit 1) (value "+5V") (footprint "")
-    )
-    (path "/00000000-0000-0000-0000-000061c840a7"
-      (reference "#PWR03") (unit 1) (value "GND") (footprint "")
-    )
     (path "/00000000-0000-0000-0000-000061c9d44f"
       (reference "#PWR04") (unit 1) (value "+5V") (footprint "")
@@
       (reference "#PWR08") (unit 1) (value "GND") (footprint "")
     )
-    (path "/00000000-0000-0000-0000-000061c836ec"
-      (reference "C1") (unit 1) (value "100nF") (footprint "Capacitors_SMD:C_0402_NoSilk")
-    )
     (path "/00000000-0000-0000-0000-000061c96815"
       (reference "D1") (unit 1) (value "WS2812B") (footprint "RGBW_LED_circular_panel_for_Stealthburner:WS2812B-2020")
@@
       (reference "J1") (unit 1) (value "Conn_02x03_Odd_Even") (footprint "Pin_Headers:Pin_Header_Straight_2x03_Pitch2.00mm_SMD")
     )
-    (path "/00000000-0000-0000-0000-000061c86569"
-      (reference "R1") (unit 1) (value "470R") (footprint "Resistors_SMD:R_0402_NoSilk")
-    )
-  )
+  )
