File: printer_mods/Mastah/breakbox_and_toolhead_pcb/KiCad/toolhead/vanilla_afterburner/toolhead_pcb.kicad_pcb (KiCad board)
At the start: 2 copper layers, 52 x 33.5 mm, 16 parts

Commit message: Update PCBs and fix some issues
Routing:
- net (no net): track 696.8 -> 698.6 mm
Other:
- board text added: "V1.2 Toolhead Design by Mastah"
- board text removed: "V1.1 Toolhead Design by Mastah"

Commit message: Update LED position
Parts:
- turned Hotend Led to 180 degrees
Other:
- board text added: "V1.3 Toolhead Design by Mastah"
- board text removed: "V1.2 Toolhead Design by Mastah"
Changed lines of the file:
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@@
   )
   (footprint "voron_led:150302RS73100" (layer "F.Cu")
-    (at 72.4 97.7)
+    (at 72.4 97.7 180)
     (attr smd)
-    (fp_text reference "Hotend Led" (at 0 1.6 unlocked) (layer "F.SilkS")
+    (fp_text reference "Hotend Led" (at 0 -1.6 unlocked) (layer "F.SilkS")
       (effects (font (size 0.6 0.6) (thickness 0.1)))
     )
-    (fp_text value "150302RS73100" (at 0 1 unlocked) (layer "F.Fab") hide
+    (fp_text value "150302RS73100" (at 0 1 180 unlocked) (layer "F.Fab") hide
       (effects (font (size 1 1) (thickness 0.15)))
     )
-    (fp_text user "+" (at -2.43 -0.07 unlocked) (layer "F.SilkS")
+    (fp_text user "+" (at -2.43 -0.07 180 unlocked) (layer "F.SilkS")
       (effects (font (size 1 1) (thickness 0.15)))
     )
-    (fp_text user "-" (at 2.46 -0.07 unlocked) (layer "F.SilkS")
+    (fp_text user "-" (at 2.46 -0.07 180 unlocked) (layer "F.SilkS")
       (effects (font (size 1 1) (thickness 0.15)))
     )
-    (fp_text user "${REFERENCE}" (at 0 2.5 unlocked) (layer "F.Fab") hide
+    (fp_text user "${REFERENCE}" (at 0 2.5 180 unlocked) (layer "F.Fab") hide
       (effects (font (size 1 1) (thickness 0.15)))
     )
@@
         (xy 0.69 0.34)
       ) (layer "F.SilkS") (width 0.02) (fill solid))
-    (pad "1" smd rect (at -1.2 0) (size 0.8 1.6) (layers "F.Cu" "F.Paste" "F.Mask"))
-    (pad "2" smd rect (at 1.2 0) (size 0.8 1.6) (layers "F.Cu" "F.Paste" "F.Mask"))
+    (pad "1" smd rect (at -1.2 0 180) (size 0.8 1.6) (layers "F.Cu" "F.Paste" "F.Mask"))
+    (pad "2" smd rect (at 1.2 0 180) (size 0.8 1.6) (layers "F.Cu" "F.Paste" "F.Mask"))
   )
   (footprint "Connector_Molex:Molex_Micro-Fit_3.0_43045-1800_2x09_P3.00mm_Horizontal" (layer "F.Cu")
@@
     (effects (font (size 0.6 0.6) (thickness 0.1)))
   )
-  (gr_text "V1.2\n\nToolhead\n\nDesign by\nMastah" (at 68.7 86.9) (layer "F.SilkS")
+  (gr_text "V1.3\n\nToolhead\n\nDesign by\nMastah" (at 68.7 86.9) (layer "F.SilkS")
     (effects (font (size 0.6 0.6) (thickness 0.1)) (justify left))
   )
