File: printer_mods/Mastah/breakbox_and_toolhead_pcb/KiCad/toolhead/stealthburner/one_pcb/toolhead_pcb.kicad_pcb (KiCad board)
At the start: 2 copper layers, 45 x 35 mm, 16 parts

Commit message: Minor placement revision
Routing:
- net (no net): track 658.3 -> 655.7 mm

Commit message: Stealthburner toolhead revision 1.1
Routing:
- net (no net): track 655.7 -> 648.9 mm
Other:
- board text added: "V1.1 Toolhead Design by Mastah"
- board text removed: "V1.0 Toolhead Design by Mastah"
