File: printer_mods/Mastah/the_bad_breath/KiCad/the_bad_breath_fan_pcb/fan_pcb/fan_pcb.kicad_pcb (KiCad board)
At the start: 2 copper layers, 28 x 15 mm, 9 parts

Commit message: Update PCB
Parts:
- removed the G*** at (32.5, 25.5)
- added G***: LOGO, voron_logo:black_hole_5x5, B.Cu at (22.9, 27.5)
- added REF**: JST_XH_S2B-XH-A-1_1x02_P2.50mm_Horizontal, Connector_JST:JST_XH_S2B-XH-A-1_1x02_P2.50mm_Horizontal, F.Cu at (32.8, 26.2)
- moved G*** 15.1 mm to (22.3, 27.4)
- moved REF** 1.55 mm to (30.2, 28.8)
Routing:
- net (no net): track 51.3 -> 65.2 mm
Other:
- board text added: "V1.1 - The Bad Breath Design by Mastah"
- board text removed: "V1.0 The Bad Breath Design by Mastah"
